Commit message: 20260917 sync from staging repo
Signed-off-by: Aaron Chong <aaronchongth@gmail.com>

File: robot_hardware_description/urdf/robot.urdf.xacro (robot description, xacro)
@@ -20,9 +20,7 @@
   <!-- Local hardware components -->
   <xacro:include
-    filename="$(find robot_hardware_description)/urdf/axia80_m20/axia80_m20_macro.xacro"/>
+    filename="$(find robot_hardware_description)/urdf/robotiq_hande/robotiq_hande_macro.xacro"/>
   <xacro:include
-    filename="$(find robot_hardware_description)/urdf/camera_mount/cam_mount_macro.xacro"/>
-  <xacro:include
-    filename="$(find robot_hardware_description)/urdf/robotiq_hande/robotiq_hande_macro.xacro"/>
+    filename="$(find robot_hardware_description)/urdf/orbbec_gemini_335le/orbbec_gemini_335le_macro.xacro"/>
   <!-- UR5e Arm -->
   <xacro:ur5e_robot
@@ -32,13 +30,10 @@
     <origin xyz="0 0 0" rpy="0 0 0"/>
   </xacro:ur5e_robot>
-  <!-- External FT sensor -->
-  <xacro:axia80_m20 tf_prefix="axia_"/>
-  <!-- Camera mounting plate -->
-  <xacro:camera_mount tf_prefix="camera_mount_"/>
-  <!-- Robotiq Hand-E -->
+  <!-- Robotiq Hand-E, adding 1mm additional opening to grasp 50mm objects -->
+  <!-- This has been reflected in third_party/robot_hardware_moveit_config/config/robot_hardware.srdf as well -->
   <xacro:robotiq_hande
     name="robotiq_hande"
     tf_prefix="hande_"
-    grip_pos_min="0.0"
+    grip_pos_min="-0.001"
     grip_pos_max="0.025"
     grip_vel_max="0.05"
@@ -47,21 +42,19 @@
     initial_pos="0.00655"
     use_ros2_control="false"/>
-  <!-- UR5e flange -> camera/FT mounting plate -->
-  <joint name="flange_to_camera_mount" type="fixed">
-    <origin xyz="0 0 -.0265" rpy="0 0 0"/>
+  <!-- Orbbec Gemini 335Le Camera -->
+  <xacro:orbbec_gemini_335le
+    name="orbbec_camera"
+    tf_prefix="orbbec_camera_"/>
+  <!-- UR5e flange -> Hand-E -->
+  <joint name="flange_to_hande" type="fixed">
+    <origin xyz="0 0 0" rpy="0 0 0"/>
     <parent link="flange"/>
-    <child link="camera_mount_cam_mount_link"/>
-  </joint>
-  <!-- Mounting plate -> Axia80-M20 -->
-  <joint name="camera_mount_to_axia80" type="fixed">
-    <origin xyz="0 0 0.0265" rpy="0 0 0"/>
-    <parent link="camera_mount_cam_mount_link"/>
-    <child link="axia_base_link"/>
-  </joint>
-  <!-- Axia80-M20 -> Hand-E -->
-  <joint name="axia80_to_hande" type="fixed">
-    <origin xyz="0 0 0" rpy="0 0 0"/>
-    <parent link="axia_tool_link"/>
     <child link="hande_hande_base_link"/>
   </joint>
+  <!-- UR5e flange -> Camera -->
+  <joint name="flange_to_orbbec_camera" type="fixed">
+    <origin xyz="0.025379 0.093008 0.077824" rpy="-0.35550899 0.00730122 3.13241238"/>
+    <parent link="flange"/>
+    <child link="orbbec_camera_link"/>
+  </joint>
 </robot>

File: robot_hardware_description/urdf/robotiq_hande/robotiq_hande_macro.xacro (robot description, xacro)
@@ -17,77 +17,66 @@
     <xacro:if value="${use_ros2_control}">
       <xacro:robotiq_hande_ros2_control
-      name="${name}"
-      tf_prefix="${tf_prefix}"
-      grip_pos_min="${grip_pos_min}"
-      grip_pos_max="${grip_pos_max}"
-      grip_effort_min="${grip_effort_min}"
-      grip_effort_max="${grip_effort_max}"
-      initial_pos="${initial_pos}"
+        name="${name}"
+        tf_prefix="${tf_prefix}"
+        grip_pos_min="${grip_pos_min}"
+        grip_pos_max="${grip_pos_max}"
+        grip_effort_min="${grip_effort_min}"
+        grip_effort_max="${grip_effort_max}"
+        initial_pos="${initial_pos}"
       />
     </xacro:if>
-    <xacro:property name="gripper_jaw_offset" value="0.025"/>
+    <!-- Base of the gripper -->
     <link name="${tf_prefix}hande_base_link">
       <inertial>
         <origin xyz="0 0 0" rpy="0 0 0"/>
         <mass value="1.0"/>
-        <inertia ixx="0.1" ixy="0" ixz="0"
-                 iyy="0.1" iyz="0"
+        <inertia ixx="0.1" ixy="0.0" ixz="0.0"
+                 iyy="0.1" iyz="0.0"
                  izz="0.1"/>
       </inertial>
-      <visual name="hande_base_visual">
+      <visual name="visual1">
         <origin xyz="0 0 0" rpy="0 0 0"/>
         <geometry>
-          <mesh filename="package://robot_hardware_description/meshes/robotiq_hande/hande_base_visual.obj"/>
+          <mesh filename="package://robot_hardware_description/meshes/robotiq_hande/robotiq_hande_body.dae"/>
         </geometry>
       </visual>
-      <collision name="body_collider_cylinder">
-        <origin xyz="0.0 0.0 0.06855" rpy="3.141593 0.0 1.570796"/>
+      <collision name="collision1">
+        <origin xyz="0 0 0" rpy="0 0 0"/>
         <geometry>
-          <cylinder radius="0.038" length="0.1131"/>
+          <mesh filename="package://robot_hardware_description/meshes/robotiq_hande/robotiq_hande_body_c01.stl"/>
         </geometry>
       </collision>
-      <collision name="cylinder003_collider_cylinder">
-        <origin xyz="0.0 0.0 0.006" rpy="0.0 0.0 0.0"/>
+      <collision name="collision2">
+        <origin xyz="0 0 0" rpy="0 0 0"/>
         <geometry>
-          <cylinder radius="0.043" length="0.012"/>
+          <mesh filename="package://robot_hardware_description/meshes/robotiq_hande/robotiq_hande_body_c02.stl"/>
         </geometry>
       </collision>
     </link>
+    <!-- Fingers and their prismatic joints -->
     <link name="${tf_prefix}hande_finger_link_l">
       <inertial>
         <origin xyz="0 0 0" rpy="0 0 0"/>
-        <mass value="0.001"/>
-        <inertia ixx="0.0001" ixy="0" ixz="0"
-                 iyy="0.00009" iyz="0"
+        <mass value="0.2"/>
+        <inertia ixx="0.0001" ixy="0.0" ixz="0.0"
+                 iyy="0.00009" iyz="0.0"
                  izz="0.00003"/>
       </inertial>
-      <visual name="hande_finger_visual">
-        <origin xyz="${-gripper_jaw_offset} 0 0" rpy="0 0 0"/>
+      <visual name="visual1">
+        <origin xyz="0 0 0" rpy="0 0 0"/>
         <geometry>
-          <mesh filename="package://robot_hardware_description/meshes/robotiq_hande/hande_finger_visual.obj"/>
+          <mesh filename="package://robot_hardware_description/meshes/robotiq_hande/robotiq_hande_finger.dae"/>
         </geometry>
       </visual>
-      <collision name="finger_collider_box">
-        <origin xyz="${-gripper_jaw_offset + 0.032595} -0.00001 0.138138" rpy="0.0 0.0 0.0"/>
+      <collision name="collision1">
+        <origin xyz="0.028 0 0.15" rpy="0 0 0"/>
         <geometry>
-          <box size="0.007839 0.021 0.028622"/>
+          <sphere radius="0.003"/>
         </geometry>
       </collision>
-      <collision name="finger_collider_box001">
-        <origin xyz="${-gripper_jaw_offset + 0.028} -0.00001 0.16145" rpy="0.0 0.0 0.0"/>
+      <collision name="collision2">
+        <origin xyz="0.033 0 0.127" rpy="0 0 0"/>
         <geometry>
-          <box size="0.006 0.021 0.021498"/>
-        </geometry>
-      </collision>
-      <collision name="finger_collider_box002">
-        <origin xyz="${-gripper_jaw_offset + 0.014354} -0.015 0.124725" rpy="0.0 0.0 0.0"/>
-        <geometry>
-          <box size="0.044319 0.0075 0.003949"/>
-        </geometry>
-      </collision>
-      <collision name="finger_collider_box003">
-        <origin xyz="${-gripper_jaw_offset + 0.027046} -0.00954 0.129064" rpy="0.0 0.0 0.0"/>
-        <geometry>
-          <box size="0.017387 0.018419 0.009271"/>
+          <box size="0.005 0.02 0.02"/>
         </geometry>
       </collision>
@@ -96,37 +85,25 @@
       <inertial>
         <origin xyz="0 0 0" rpy="0 0 0"/>
-        <mass value="0.001"/>
-        <inertia ixx="0.0001" ixy="0" ixz="0"
-                 iyy="0.00009" iyz="0"
+        <mass value="0.2"/>
+        <inertia ixx="0.0001" ixy="0.0" ixz="0.0"
+                 iyy="0.00009" iyz="0.0"
                  izz="0.00003"/>
       </inertial>
-      <visual name="hande_finger_visual">
-        <origin xyz="${gripper_jaw_offset} 0 0" rpy="0 0 3.14157"/>
+      <visual name="visual1">
+        <origin xyz="0 0 0" rpy="0 0 3.14157"/>
         <geometry>
-          <mesh filename="package://robot_hardware_description/meshes/robotiq_hande/hande_finger_visual.obj"/>
+          <mesh filename="package://robot_hardware_description/meshes/robotiq_hande/robotiq_hande_finger.dae"/>
         </geometry>
       </visual>
-      <collision name="finger_collider_box">
-        <origin xyz="${gripper_jaw_offset - 0.032595} -0.00001 0.138138" rpy="0.0 0.0 0.0"/>
+      <collision name="collision1">
+        <origin xyz="-0.028 0 0.15" rpy="0 0 0"/>
         <geometry>
-          <box size="0.007839 0.021 0.028622"/>
+          <sphere radius="0.003"/>
         </geometry>
       </collision>
-      <collision name="finger_collider_box001">
-        <origin xyz="${gripper_jaw_offset - 0.028} -0.00001 0.16145" rpy="0.0 0.0 0.0"/>
+      <collision name="collision2">
+        <origin xyz="-0.033 0 0.127" rpy="0 0 0"/>
         <geometry>
-          <box size="0.006 0.021 0.021498"/>
-        </geometry>
-      </collision>
-      <collision name="finger_collider_box002">
-        <origin xyz="${gripper_jaw_offset - 0.014354} -0.015 0.124725" rpy="0.0 0.0 0.0"/>
-        <geometry>
-          <box size="0.044319 0.0075 0.003949"/>
-        </geometry>
-      </collision>
-      <collision name="finger_collider_box003">
-        <origin xyz="${gripper_jaw_offset - 0.027046} -0.00954 0.129064" rpy="0.0 0.0 0.0"/>
-        <geometry>
-          <box size="0.017387 0.018419 0.009271"/>
+          <box size="0.005 0.02 0.02"/>
         </geometry>
       </collision>
@@ -136,5 +113,5 @@
       <parent link="${tf_prefix}hande_base_link"/>
       <child link="${tf_prefix}hande_finger_link_l"/>
-      <axis xyz="1 0 0"/>
+      <axis xyz="-1 0 0"/>
       <limit effort="${grip_effort_max}" lower="${grip_pos_min}" upper="${grip_pos_max}" velocity="${grip_vel_max}"/>
     </joint>
@@ -143,15 +120,17 @@
       <parent link="${tf_prefix}hande_base_link"/>
       <child link="${tf_prefix}hande_finger_link_r"/>
-      <axis xyz="-1 0 0"/>
+      <axis xyz="1 0 0"/>
       <limit effort="${grip_effort_max}" lower="${grip_pos_min}" upper="${grip_pos_max}" velocity="${grip_vel_max}"/>
       <mimic joint="${tf_prefix}left_finger_joint" multiplier="1" offset="0"/>
     </joint>
+    <!-- Tool Center Point (TCP) and Tool Frame conventions -->
     <link name="${tf_prefix}tcp"/>
     <joint name="${tf_prefix}attach_tool_frame" type="fixed">
-      <origin xyz="0 0 0.172" rpy="0 0 0"/>
+    <!-- NOTE(aaronchongth): decreased z-offset from 0.172 to 0.14 because of constant collisions with scene objects -->
+      <origin xyz="0 0 0.14" rpy="0 0 0"/>
       <parent link="${tf_prefix}hande_base_link"/>
       <child link="${tf_prefix}tcp"/>
     </joint>
-    <!-- Alias link for Flowstate prefixed tool_frame convention -->
+    <!-- Alias link for Intrinsic Core prefixed tool_frame convention -->
     <link name="${tf_prefix}tool_frame"/>
     <joint name="${tf_prefix}tcp_to_prefixed_tool_frame" type="fixed">
@@ -160,5 +139,5 @@
       <child link="${tf_prefix}tool_frame"/>
     </joint>
-    <!-- Alias link for Flowstate unqualified tool_frame convention -->
+    <!-- Alias link for Intrinsic Core unqualified tool_frame convention -->
     <link name="tool_frame"/>
     <joint name="${tf_prefix}tcp_to_tool_frame" type="fixed">
@@ -167,4 +146,11 @@
       <child link="tool_frame"/>
     </joint>
+    <!-- Alias link for Intrinsic Core gripper base convention -->
+    <link name="gripper_base_link"/>
+    <joint name="${tf_prefix}base_to_gripper_base_link" type="fixed">
+      <origin xyz="0 0 0" rpy="0 0 0"/>
+      <parent link="${tf_prefix}hande_base_link"/>
+      <child link="gripper_base_link"/>
+    </joint>
   </xacro:macro>
 </robot>

File: robot_hardware_description/urdf/ur5e/ur5e.urdf (robot description, URDF)
Before this commit: robot ur5e, 7 links, 6 joints
Joints:
- joint wrist_3_joint: origin xyz=0.0 0.0996 0 rpy=-1.57079632679 0 0 -> xyz=0.0 0.0996 0 rpy=-1.57079632679 3.14159265359 0

File: robot_hardware_description/urdf/ur5e/ur5e_macro.xacro (robot description, xacro)
@@ -23,7 +23,13 @@
       </visual>
       <collision>
-        <origin rpy="0 0 3.14159265359" xyz="0 0 0"/>
-        <geometry>
-          <mesh filename="package://robot_hardware_description/urdf/ur5e/collision/base.wrapped.1cm.stl"/>
+        <!--
+          TODO(aaronchongth): we use the non-inflated base collision, as well as raising the
+          collision by 1cm, to prevent base collision with the mount. This should be revisited and
+          fixed when we start using upstream URDFs.
+        -->
+        <origin rpy="0 0 3.14159265359" xyz="0 0 0.01"/>
+        <geometry>
+          <!-- <mesh filename="package://robot_hardware_description/urdf/ur5e/collision/base.wrapped.1cm.stl"/> -->
+          <mesh filename="package://robot_hardware_description/urdf/ur5e/collision/base.stl"/>
         </geometry>
       </collision>
@@ -181,5 +187,5 @@
       <parent link="${tf_prefix}wrist_2_link"/>
       <child link="${tf_prefix}wrist_3_link"/>
-      <origin rpy="-1.57079632679 0 0" xyz="0.0 0.0996 0"/>
+      <origin rpy="-1.57079632679 3.14159265359 0" xyz="0.0 0.0996 0"/>
       <axis xyz="0 0 1"/>
       <limit effort="28.0" lower="-6.2831853" upper="6.2831853" velocity="3.1415927"/>
